File: ELI2040.kicad_pcb (KiCad board)
At the start: 2 copper layers, 23.8 x 83.4 mm, 50 parts, among them J15 SWD, J2 Power Header, J3 ADCs Header, J4 Conn_01x26, J7 Conn_02x01, J8 Conn_02x01, U1 TLV76733DRVR, U11 W25Q128JVS, U4 TLV76733DRVR, U7 RP2040, Y1 YXC X322512MSB4SI

Commit message: update 2
Parts:
- removed FB2: FerriteBead GZ2012D101TF, Resistor_SMD:R_0805_2012Metric
- removed R1, R2: 5.1k, Resistor_SMD:R_0402_1005Metric
- removed USB1: MC-110LS-L100, emutelab:TYPE-C-SMD_GT-USB-7082D
- added D1: 1N5819, Diode_SMD:D_SOD-323, F.Cu at (215.4, 43.9)
- added J1: GND1, Connector_PinHeader_2.54mm:PinHeader_1x02_P2.54mm_Vertical, F.Cu at (208.3, 121.9)
- added J5: GND2, Connector_PinHeader_2.54mm:PinHeader_1x02_P2.54mm_Vertical, F.Cu at (208.3, 38.1)
- added R3: 5.1k, Resistor_SMD:R_0402_1005Metric, F.Cu at (154.5, 31.7)
- added R4: 5.1k, Resistor_SMD:R_0402_1005Metric, F.Cu at (154.5, 33.7)
- added USB2: TYPE-C_16PIN_2MD(073), emutelab:USB-C-SMD_TYPE-C-6PIN-2MD-073, F.Cu at (211.0, 47.8)
- J3: footprint Connector_PinHeader_2.54mm:PinHeader_1x05_P2.54mm_Vertical -> Connector_PinHeader_2.54mm:PinHeader_1x06_P2.54mm_Vertical
- J4: footprint Connector_PinHeader_2.54mm:PinHeader_1x26_P2.54mm_Vertical -> Connector_PinHeader_2.54mm:PinHeader_1x27_P2.54mm_Vertical
- TP8: moved to F.Cu
- moved R31 158.8 mm to (218.9, 121.9)
- moved R37 155.3 mm to (215.8, 121.9), turned to 0 degrees
- moved J8 150.1 mm to (215.9, 119.4)
- moved J7 149.6 mm to (215.9, 124.5)
- moved TP2 54.4 mm to (147.3, 83.8)
- moved C3 53.3 mm to (218.4, 38.5)
- moved D4 52.1 mm to (220.6, 38.4)
- moved C27 52.0 mm to (216.2, 79.6), turned to -135 degrees
- moved Y1 51.9 mm to (216.5, 82.4), turned to 45 degrees
- moved C28 51.4 mm to (219.7, 81.2), turned to 45 degrees
- moved C20 51.4 mm to (210.5, 79.5), turned to -135 degrees
- moved C8 50.9 mm to (219.7, 49.2), turned to 0 degrees
- moved R36 50.2 mm to (219.2, 79.9), turned to -135 degrees
- moved C21 49.2 mm to (218.1, 78.2), turned to 0 degrees
- moved C18 49.2 mm to (208.0, 76.1), turned to 135 degrees
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Connections:
- D4 pad 2: Net-(D4-A) -> 12V_IN
- J4 pad 1: /GPIO0 -> GND
- J4 pad 10: /GPIO11 -> /GPIO9
- J4 pad 11: /GPIO12 -> /GPIO10
- J4 pad 12: /GPIO13 -> /GPIO11
- J4 pad 13: /GPIO14 -> /GPIO12
- J4 pad 14: /GPIO15 -> /GPIO13
- J4 pad 15: /GPIO16 -> /GPIO14
- J4 pad 16: /GPIO17 -> /GPIO15
- J4 pad 17: /GPIO18 -> /GPIO16
- J4 pad 18: /GPIO19 -> /GPIO17
- J4 pad 19: /GPIO20 -> /GPIO18
- J4 pad 2: /GPIO2 -> +3V3
- J4 pad 20: /GPIO21 -> /GPIO19
- J4 pad 21: /GPIO23 -> /GPIO20
- J4 pad 22: /GPIO24 -> /GPIO21
- J4 pad 23: /GPIO25 -> /GPIO23
- J4 pad 24: /BOOTSEL -> /GPIO24
- J4 pad 25: /RUN -> /GPIO25
- J4 pad 26: GND -> /BOOTSEL
- J4 pad 3: /GPIO3 -> /GPIO0
- J4 pad 4: /GPIO5 -> /GPIO2
- J4 pad 5: /GPIO6 -> /GPIO3
- J4 pad 6: /GPIO7 -> /GPIO5
- J4 pad 7: /GPIO8 -> /GPIO6
- J4 pad 8: /GPIO9 -> /GPIO7
- J4 pad 9: /GPIO10 -> /GPIO8
Routing:
- net /GPIO4_SDA: track 0.00 -> 58.4 mm, vias 0 -> 1
- net /GPIO1_SCL: track 0.00 -> 53.9 mm, vias 0 -> 1
- net /GPIO0: track 0.00 -> 51.9 mm
- net /GPIO2: track 0.55 -> 48.4 mm
- net /GPIO3: track 0.00 -> 45.4 mm
- net /GPIO5: track 0.00 -> 41.5 mm
- net /GPIO6: track 0.00 -> 38.6 mm
- net /GPIO7: track 0.00 -> 35.7 mm
- net /+3V3_SIG: track 38.2 -> 2.83 mm
- net /GPIO8: track 0.00 -> 31.5 mm
- net /GPIO9: track 0.00 -> 28.6 mm
- net /GPIO13: track 0.00 -> 28.2 mm
- net /GPIO10: track 0.00 -> 25.6 mm
- net /GPIO11: track 0.00 -> 22.9 mm
- net /GPIO12: track 0.00 -> 21.5 mm
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- removed copper zone on F.Cu, net (none)
Other:
- board size 23.8 x 83.4 mm -> 19.9 x 90.4 mm

Commit message: update 3
Parts:
- moved R65 141.4 mm to (220.0, 87.6), turned to 180 degrees
- moved D15 140.2 mm to (220.0, 89.2), turned to 180 degrees
- moved R4 63.0 mm to (215.2, 50.6), turned to -45 degrees
- moved R3 62.4 mm to (215.2, 46.4)
- moved R30 58.1 mm to (209.1, 55.4)
- moved R29 55.7 mm to (207.0, 57.6), turned to 0 degrees
- moved C33 54.8 mm to (214.2, 55.2)
- moved TP1 8.53 mm to (97.3, 34.2)
- moved C37 0.79 mm to (215.1, 68.1)
- moved R22 0.65 mm to (211.6, 68.7), turned to -135 degrees
- moved C3 0.28 mm to (218.5, 38.2)
- moved C1 0.10 mm to (211.3, 39.5)
- moved C2 0.10 mm to (216.1, 40.1)
- moved U1 0.10 mm to (213.6, 40.0)
Routing:
- net +3V3: track 43.0 -> 73.7 mm
- net /USB_D-: track 0.00 -> 28.2 mm
- net /USB_D+: track 0.00 -> 26.6 mm
- net /+3V3_SIG: track 2.83 -> 24.5 mm
- net /GPIO22_TEST_LED: track 3.67 -> 23.1 mm, vias 0 -> 2
- net +12V: track 25.6 -> 38.0 mm
- net GND: track 16.2 -> 19.0 mm, vias 17 -> 19
- net /GPIO14: track 19.7 -> 21.5 mm
- net Net-(USB2-CC2): track 0.00 -> 1.77 mm
- net Net-(D15-A): track 0.00 -> 1.63 mm
- net Net-(USB2-CC1): track 0.00 -> 1.36 mm
- net /GPIO18: track 8.61 -> 7.67 mm

Commit message: latest v0.1
Parts:
- removed J15: SWD, Connector_PinHeader_2.54mm:PinHeader_1x03_P2.54mm_Vertical
- removed S1, S2: B3U-1000P, digikey-footprints:Switch_Tactile_SMD_B3U-1000P
- removed TP1: RP2040 Power, TestPoint:TestPoint_Pad_1.5x1.5mm
- removed TP2: Analog Power, TestPoint:TestPoint_Pad_1.5x1.5mm
- removed TP8: 1V1, TestPoint:TestPoint_Pad_1.5x1.5mm
- added C4: 100n, Capacitor_SMD:C_0402_1005Metric, F.Cu at (207.0, 55.9)
- added C6: 100n, Capacitor_SMD:C_0402_1005Metric, F.Cu at (221.2, 121.8)
- added SW1: TS-1187A-B-A-B, emutelab:SW-SMD_4P-L5.1-W5.1-P3.70-LS6.5-TL-2, F.Cu at (210.6, 107.9)
- added SW2: TS-1187A-B-A-B, emutelab:SW-SMD_4P-L5.1-W5.1-P3.70-LS6.5-TL-2, F.Cu at (210.6, 114.3)
- R30: footprint Capacitor_SMD:C_0805_2012Metric -> Capacitor_SMD:C_01005_0402Metric
- moved R29 1.52 mm to (207.6, 59.0), turned to 45 degrees
- moved R30 1.22 mm to (210.2, 56.0), turned to -135 degrees
- moved C33 0.54 mm to (213.9, 55.7), turned to -45 degrees
Connections:
- U7 pad 24: /SWCLK -> unconnected-(U7-SWCLK-Pad24)
- U7 pad 25: /SWD -> unconnected-(U7-SWD-Pad25)
Routing:
- net +3V3: track 73.7 -> 207.6 mm, vias 0 -> 3
- net /BOOTSEL: track 0.00 -> 75.3 mm, vias 0 -> 3
- net /RUN: track 1.81 -> 63.1 mm, vias 1 -> 2
- net /QSPI_SS: track 15.8 -> 25.9 mm
- net /+3V3_SIG: track 24.5 -> 34.1 mm, vias 0 -> 2
- net /VBUS: track 2.11 -> 8.45 mm
- net GND: track 19.0 -> 25.2 mm, vias 19 -> 43
- net /SWCLK: track 3.58 -> 0.00 mm
- net /GPIO0: track 51.9 -> 54.6 mm
- net /USB_D+: track 26.6 -> 28.7 mm
- net +12V: track 38.0 -> 40.0 mm, vias 2 -> 4
- net /GPIO2: track 48.4 -> 49.7 mm
- net /GPIO29_ADC3: track 27.5 -> 26.7 mm
- net /USB_D-: track 28.2 -> 28.9 mm
- net /GPIO25: track 11.8 -> 12.4 mm
Other:
- board text added: "ELI2040 v0.1a Emute Lab Instruments 2024"
- board text removed: "GND"
- board text removed: "SWCLK"
- board text removed: "SWD"
