File: ELI2040.kicad_sch (KiCad schematic)
At the start: 50 parts, among them J15 SWD, J2 Power Header, J3 ADCs Header, J4 Conn_01x26, J7 Conn_02x01, J8 Conn_02x01, U1 TLV76733DRVR, U11 W25Q128JVS, U4 TLV76733DRVR, U7 RP2040, Y1 YXC X322512MSB4SI

Commit message: update 2
Parts:
- removed FB2: FerriteBead GZ2012D101TF, Resistor_SMD:R_0805_2012Metric, symbol Device:FerriteBead
- removed R1, R2: 5.1k, Resistor_SMD:R_0402_1005Metric, symbol Device:R
- removed USB1: MC-110LS-L100, emutelab:TYPE-C-SMD_GT-USB-7082D, symbol emutelab:MC-110LS-L100
- added D1: 1N5819, Diode_SMD:D_SOD-323, symbol Diode:1N5818
- added J1: GND1, Connector_PinHeader_2.54mm:PinHeader_1x02_P2.54mm_Vertical, symbol Connector_Generic:Conn_01x02
- added J5: GND2, Connector_PinHeader_2.54mm:PinHeader_1x02_P2.54mm_Vertical, symbol Connector_Generic:Conn_01x02
- added R3, R4: 5.1k, Resistor_SMD:R_0402_1005Metric, symbol Device:R
- added USB2: TYPE-C_16PIN_2MD(073), emutelab:USB-C-SMD_TYPE-C-6PIN-2MD-073, symbol emutelab:TYPE-C_16PIN_2MD(073)
- J3: footprint Connector_PinHeader_2.54mm:PinHeader_1x05_P2.54mm_Vertical -> Connector_PinHeader_2.54mm:PinHeader_1x06_P2.54mm_Vertical
- J4: footprint Connector_PinHeader_2.54mm:PinHeader_1x26_P2.54mm_Vertical -> Connector_PinHeader_2.54mm:PinHeader_1x27_P2.54mm_Vertical
Connections:
- net +12V: now also D1.1 (K)
- net 12V_IN: now also D4.2 (A)
- net BOOTSEL: now also J4.26 (Pin_26); no longer J4.3 (Pin_3)
- net GND: now also J1.1 (Pin_1), J1.2 (Pin_2), J5.1 (Pin_1), J5.2 (Pin_2), R3.2, R4.2, USB2.1 (GND), USB2.12 (GND), USB2.13 (SHELL), USB2.14 (SHELL)
- net GPIO0: now also J4.3 (Pin_3); no longer J4.5 (Pin_5)
- net GPIO10: now also J4.11 (Pin_11); no longer J4.13 (Pin_13)
- net GPIO11: now also J4.12 (Pin_12); no longer J4.14 (Pin_14)
- net GPIO12: now also J4.13 (Pin_13); no longer J4.15 (Pin_15)
- net GPIO13: now also J4.14 (Pin_14); no longer J4.16 (Pin_16)
- net GPIO14: now also J4.15 (Pin_15); no longer J4.17 (Pin_17)
- net GPIO15: now also J4.16 (Pin_16); no longer J4.18 (Pin_18)
- net GPIO16: now also J4.17 (Pin_17); no longer J4.19 (Pin_19)
- net GPIO17: now also J4.18 (Pin_18); no longer J4.20 (Pin_20)
- net GPIO18: now also J4.19 (Pin_19); no longer J4.21 (Pin_21)
- net GPIO19: now also J4.20 (Pin_20); no longer J4.22 (Pin_22)
- net GPIO2: now also J4.4 (Pin_4); no longer J4.6 (Pin_6)
- net GPIO20: now also J4.21 (Pin_21); no longer J4.23 (Pin_23)
- net GPIO21: now also J4.22 (Pin_22); no longer J4.24 (Pin_24)
- net GPIO23: now also J4.23 (Pin_23); no longer J4.25 (Pin_25)
- net GPIO24: now also J4.24 (Pin_24); no longer J4.26 (Pin_26)
- net GPIO25: now also J4.25 (Pin_25); no longer J4.27 (Pin_27)
- net GPIO3: now also J4.5 (Pin_5); no longer J4.7 (Pin_7)
- net GPIO5: now also J4.6 (Pin_6); no longer J4.8 (Pin_8)
- net GPIO6: now also J4.7 (Pin_7); no longer J4.9 (Pin_9)
- net GPIO7: now also J4.8 (Pin_8); no longer J4.10 (Pin_10)
- net GPIO8: now also J4.9 (Pin_9); no longer J4.11 (Pin_11)
- net GPIO9: now also J4.10 (Pin_10); no longer J4.12 (Pin_12)
- net RUN: now also J4.27 (Pin_27); no longer J4.4 (Pin_4)
- net USB_D+: now also USB2.6 (DP1), USB2.8 (DP2)
- net USB_D-: now also USB2.5 (DN2), USB2.7 (DN1)
- new net: R3.1, USB2.4 (CC1)
- new net: R4.1, USB2.10 (CC2)
- new net VBUS: D1.2 (A), USB2.11 (VBUS), USB2.2 (VBUS)
- no-connect marks 7 -> 3
Other:
- note added: "try TS-1187A-B-A-B JLC"
- moved on the sheet: J2

Commit message: update 3
Changed lines of the file:
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@@
 	)
 	(label "AGND"
-		(at 300.99 335.28 270)
+		(at 317.5 246.38 270)
 		(fields_autoplaced yes)
 		(effects
@@
 		(lib_name "GND_1")
 		(lib_id "power:GND")
-		(at 300.99 335.28 180)
+		(at 317.5 246.38 180)
 		(unit 1)
 		(exclude_from_sim no)
@@
 		(fields_autoplaced yes)
 		(property "Reference" "#PWR08"
-			(at 300.99 328.93 0)
+			(at 317.5 240.03 0)
 			(effects
 				(font
@@
 		)
 		(property "Value" "GND"
-			(at 300.99 330.2 0)
+			(at 317.5 241.3 0)
 			(effects
 				(font
@@
 		)
 		(property "Footprint" ""
-			(at 300.99 335.28 0)
+			(at 317.5 246.38 0)
 			(effects
 				(font
@@
 		)
 		(property "Datasheet" ""
-			(at 300.99 335.28 0)
+			(at 317.5 246.38 0)
 			(effects
 				(font
@@
 		)
 		(property "Description" "Power symbol creates a global label with name \"GND\" , ground"
-			(at 300.99 335.28 0)
+			(at 317.5 246.38 0)
 			(effects
 				(font

Commit message: latest v0.1
Parts:
- removed J15: SWD, Connector_PinHeader_2.54mm:PinHeader_1x03_P2.54mm_Vertical, symbol Connector_Generic:Conn_01x03
- removed S1, S2: B3U-1000P, digikey-footprints:Switch_Tactile_SMD_B3U-1000P, symbol dk_Tactile-Switches:B3U-1000P
- removed TP1: RP2040 Power, TestPoint:TestPoint_Pad_1.5x1.5mm, symbol Connector:TestPoint_Probe
- removed TP2: Analog Power, TestPoint:TestPoint_Pad_1.5x1.5mm, symbol Connector:TestPoint_Probe
- removed TP8: 1V1, TestPoint:TestPoint_Pad_1.5x1.5mm, symbol Connector:TestPoint_Probe
- added C4, C6: 100n, Capacitor_SMD:C_0402_1005Metric, symbol Device:C
- added SW1, SW2: TS-1187A-B-A-B, emutelab:SW-SMD_4P-L5.1-W5.1-P3.70-LS6.5-TL-2, symbol emutelab:TS-1187A-B-A-B
- R30: footprint Capacitor_SMD:C_0805_2012Metric -> Capacitor_SMD:C_01005_0402Metric
Connections:
- net +3V3: now also C4.1, C6.1
- net BOOTSEL: now also SW2.2 (B)
- net GND: now also C4.2, C6.2, SW1.3 (C), SW1.4 (D), SW2.3 (C), SW2.4 (D)
- net RUN: now also SW1.2 (B)
- net SWCLK: no longer names the net of U7.24 (SWCLK)
- net SWD: no longer names the net of U7.25 (SWD)
- no-connect marks 3 -> 5
Other:
- note removed: "try TS-1187A-B-A-B JLC"
- moved on the sheet: C5, C8, U4
